File: CNC.kicad_sch (KiCad schematic)
At the start: 20 parts, among them J1 Conn_01x02_Male, J2 Conn_01x01_Male, J3 SD-MODULE, J4 Micro_SD_Card, J5 UART0, J6 EXTRA1, U1 LM7805_TO220, U2 ESP32_DEVKITV1

Commit message: Added I/O Expander and fixed DRC
Parts:
- removed J6: EXTRA1, Connector_PinHeader_2.54mm:PinHeader_1x04_P2.54mm_Vertical, symbol Connector:Conn_01x04_Male
- added C16: 100nF, Capacitor_SMD:C_0805_2012Metric_Pad1.18x1.45mm_HandSolder, symbol Device:C
- added J6, J7: Conn_02x08_Odd_Even, Connector_IDC:IDC-Header_2x08_P2.54mm_Vertical, symbol Connector_Generic:Conn_02x08_Odd_Even
- added J8: I2C, Connector:FanPinHeader_1x03_P2.54mm_Vertical, symbol Connector_Generic:Conn_01x03
- added R4, R5: 4k7, Resistor_SMD:R_0805_2012Metric_Pad1.20x1.40mm_HandSolder, symbol Device:R
- added U7: MCP23017_SS, Package_SO:SSOP-28_5.3x10.2mm_P0.65mm, symbol Interface_Expansion:MCP23017_SS
Connections:
- net +3V3: now also R4.1, R5.1
- net +5V: now also C16.1, U7.18 (~{RESET}), U7.9 (VDD)
- net GND: now also C16.2, J6.10 (Pin_10), J6.12 (Pin_12), J6.14 (Pin_14), J6.16 (Pin_16), J6.2 (Pin_2), J6.4 (Pin_4), J6.6 (Pin_6), J6.8 (Pin_8), J7.10 (Pin_10), J7.12 (Pin_12), J7.14 (Pin_14), J7.16 (Pin_16), J7.2 (Pin_2), J7.4 (Pin_4), J7.6 (Pin_6), J7.8 (Pin_8), J8.3 (Pin_3), U7.10 (VSS), U7.15 (A0), U7.16 (A1), U7.17 (A2)
- net X-DIR: now also U2.20 (GPIO4/ADC2_CH0/TOUCH0); no longer U2.29 (GPIO22/I2C_SCL)
- net X-STEP: now also U2.19 (GPIO2/ADC2_CH2/TOUCH2/BOARD_LED); no longer U2.26 (GPIO21/I2C_SDA)
- new net: J6.15 (Pin_15), U7.1 (GPB0)
- new net: J6.13 (Pin_13), U7.2 (GPB1)
- new net: J7.15 (Pin_15), U7.21 (GPA0)
- new net: J7.13 (Pin_13), U7.22 (GPA1)
- new net: J7.11 (Pin_11), U7.23 (GPA2)
- new net: J7.9 (Pin_9), U7.24 (GPA3)
- new net: J7.7 (Pin_7), U7.25 (GPA4)
- new net: J7.5 (Pin_5), U7.26 (GPA5)
- new net: J7.3 (Pin_3), U7.27 (GPA6)
- new net: J7.1 (Pin_1), U7.28 (GPA7)
- new net: J6.11 (Pin_11), U7.3 (GPB2)
- new net: J6.9 (Pin_9), U7.4 (GPB3)
- new net: J6.7 (Pin_7), U7.5 (GPB4)
- new net: J6.5 (Pin_5), U7.6 (GPB5)
- new net: J6.3 (Pin_3), U7.7 (GPB6)
- new net: J6.1 (Pin_1), U7.8 (GPB7)
- new net I2C-SCL: J8.1 (Pin_1), R4.2, U2.29 (GPIO22/I2C_SCL), U7.12 (SCK)
- new net I2C-SDA: J8.2 (Pin_2), R5.2, U2.26 (GPIO21/I2C_SDA), U7.13 (SDA)
- no-connect marks 3 -> 6
Other:
- moved on the sheet: J3, J4
