File: drivers.kicad_sch (KiCad schematic)
At the start: 20 parts, among them U3 Z - TMC2209 BTT v1.2, U4 X - TMC2209 BTT v1.2, U5 A - TMC2209 BTT v1.2, U6 Y - TMC2209 BTT v1.2

Commit message: Added I/O Expander and fixed DRC
Connections:
- net MOT-UART: now also U3.5 (PDN), U4.5 (PDN), U5.5 (PDN), U6.5 (PDN)
- no-connect marks 8 -> 4
Changed lines of the file:
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@@
   (junction (at 166.37 118.11) (diameter 0) (color 0 0 0 0)
   )
+  (junction (at 49.53 110.49) (diameter 0) (color 0 0 0 0)
+  )
+  (junction (at 138.43 62.23) (diameter 0) (color 0 0 0 0)
+  )
   (junction (at 179.07 55.88) (diameter 0) (color 0 0 0 0)
   )
@@
   (junction (at 99.06 54.61) (diameter 0) (color 0 0 0 0)
   )
+  (junction (at 132.08 110.49) (diameter 0) (color 0 0 0 0)
+  )
   (junction (at 83.82 118.11) (diameter 0) (color 0 0 0 0)
   )
@@
   (junction (at 99.06 43.18) (diameter 0) (color 0 0 0 0)
   )
+  (junction (at 58.42 60.96) (diameter 0) (color 0 0 0 0)
+  )
   (junction (at 132.08 106.68) (diameter 0) (color 0 0 0 0)
   )
@@
   )
   (no_connect (at 148.59 48.26))
-  (no_connect (at 138.43 64.77))
   (no_connect (at 68.58 46.99))
-  (no_connect (at 58.42 63.5))
-  (no_connect (at 132.08 113.03))
   (no_connect (at 142.24 96.52))
   (no_connect (at 59.69 96.52))
-  (no_connect (at 49.53 113.03))
   (wire (pts (xy 58.42 57.15) (xy 58.42 58.42))
     (stroke (width 0) (type default) (color 0 0 0 0))
   )
+  (wire (pts (xy 49.53 110.49) (xy 49.53 113.03))
+    (stroke (width 0) (type default) (color 0 0 0 0))
+  )
   (wire (pts (xy 72.39 120.65) (xy 77.47 120.65))
     (stroke (width 0) (type default) (color 0 0 0 0))
@@
     (stroke (width 0) (type default) (color 0 0 0 0))
   )
+  (wire (pts (xy 132.08 110.49) (xy 132.08 113.03))
+    (stroke (width 0) (type default) (color 0 0 0 0))
+  )
   (wire (pts (xy 160.02 127) (xy 162.56 127))
     (stroke (width 0) (type default) (color 0 0 0 0))
@@
     (stroke (width 0) (type default) (color 0 0 0 0))
   )
+  (wire (pts (xy 58.42 60.96) (xy 58.42 63.5))
+    (stroke (width 0) (type default) (color 0 0 0 0))
+  )
   (wire (pts (xy 77.47 120.65) (xy 77.47 127))
     (stroke (width 0) (type default) (color 0 0 0 0))
@@
     (stroke (width 0) (type default) (color 0 0 0 0))
   )
+  (wire (pts (xy 138.43 64.77) (xy 138.43 62.23))
+    (stroke (width 0) (type default) (color 0 0 0 0))
+  )
